File: hardware/project/ICE40PROG/ICE40PROG.kicad_pcb (KiCad board)
At the start: 2 copper layers, 46 parts, among them J1 Conn_02x05, J2 USB_B_Micro, U1 LT1762-3.3, U2 FT2232H, U3 93LC56-SO8, U4 CA25C1204GLT

Commit message: Schematic, PCB and BOM done.
Parts:
- removed D1: SMBJ6.0CA, ICE40PROG:DO_214AA
- removed the R2 at (162.7, 75.2)
- removed U4: CA25C1204GLT, ICE40PROG:CA25
- added Q1: CA25C1204GLT, ICE40PROG:CA25, B.Cu at (150.0, 71.9)
- added R1: DNP, Resistor_SMD:R_0603_1608Metric_Pad1.05x0.95mm_HandSolder, F.Cu at (163.8, 63.0)
- C1, C10, C11, C12, C13, C14, C18, C2, C3, C4, C5, C6, C7, C8, C9, R10, R17, R18: moved to B.Cu
- FB1: moved to F.Cu
- J1: footprint Connector_PinSocket_2.54mm:PinSocket_2x05_P2.54mm_Horizontal -> Connector_PinSocket_2.54mm:PinSocket_2x05_P2.54mm_Vertical; moved to B.Cu
- R2: renamed from R3; moved to B.Cu
- R7: renamed from R1; value 220 -> 270
- moved C1 47.3 mm to (161.3, 71.5)
- moved C9 46.3 mm to (161.3, 66.9)
- moved R10 37.5 mm to (161.3, 70.0)
- moved D2 36.7 mm to (140.7, 67.4)
- moved C13 36.4 mm to (146.9, 67.3), turned to 90 degrees
- moved R7 35.9 mm to (144.0, 67.4)
- moved C18 35.8 mm to (152.1, 66.5), turned to 90 degrees
- moved C11 35.0 mm to (149.1, 66.5), turned to 270 degrees
- moved R2 33.7 mm to (134.1, 68.3), turned to 180 degrees
- moved C4 33.3 mm to (138.8, 66.9)
- moved C14 33.2 mm to (146.9, 63.9), turned to 90 degrees
- moved C2 31.2 mm to (161.3, 73.0)
- moved R18 29.0 mm to (153.4, 71.8), turned to 90 degrees
- moved C8 26.4 mm to (161.3, 68.5)
- moved R17 25.8 mm to (143.6, 71.9), turned to 90 degrees
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- renumbered R4 to R3, R5 to R4, R6 to R5, R7 to R6
Routing:
- net (no net): track 0.00 -> 81.8 mm
- net +3V3: track 0.00 -> 44.3 mm, vias 0 -> 17
- net +1V8: track 0.00 -> 29.1 mm, vias 0 -> 4
- net /DP: track 0.00 -> 15.3 mm, vias 0 -> 2
- net /DM: track 0.00 -> 14.4 mm, vias 0 -> 2
- net Net-(R10-Pad1): track 0.00 -> 12.4 mm, vias 0 -> 1
- net Net-(R13-Pad2): track 0.00 -> 11.7 mm
- net Net-(R12-Pad2): track 0.00 -> 11.2 mm
- net GND: track 0.00 -> 9.37 mm, vias 0 -> 7
- net Net-(R6-Pad2): track 0.00 -> 9.03 mm, vias 0 -> 2
- net Net-(R14-Pad2): track 0.00 -> 8.75 mm, vias 0 -> 1
- net Net-(R5-Pad2): track 0.00 -> 8.48 mm
- net Net-(J2-Pad2): track 0.00 -> 8.26 mm
- net Net-(R15-Pad2): track 0.00 -> 8.25 mm, vias 0 -> 1
- net Net-(R3-Pad2): track 0.00 -> 7.06 mm
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- added copper zone on B.Cu, net +3V3
- added copper zone on F.Cu, net +3V3
- added copper zone on Power, net +3V3
- added copper zone on B.Cu, net +5V
- added copper zone on F.Cu, net +5V
- added copper zone on Power, net +5V
- added copper zone on B.Cu, net GND
- added copper zone on F.Cu, net GND
- added copper zone on GND, net GND
- added copper zone on B.Cu, net GNDS
- added copper zone on F.Cu, net GNDS
- added copper zone on GND, net GNDS
- added copper zone on B.Cu, net Net-(C3-Pad1)
- added copper zone on F.Cu, net Net-(C3-Pad1)
- added copper zone on Power, net Net-(C3-Pad1)
Other:
- board outline added: 45.1 x 15 mm
- copper layers 2 -> 4
- net class Default: clearance 0.2 -> 0.127; trace_width 0.25 -> 0.127; via_dia 0.8 -> 0.5; via_drill 0.4 -> 0.2
- rule trace_clearance: 0.2 -> 0.127
- rule trace_min: 0.2 -> 0.1
- rule via_min_drill: 0.3 -> 0.2
- board text added: "1"
- board text added: "2"
- board text added: "3"
- board text added: "4"
- board text added: "iCE40PROG V1.0"
