File: hardware/project/ICE40PROG/ICE40PROG.sch (KiCad schematic (older format))
At the start: 46 parts, among them J1 Conn_02x05, J2 USB_B_Micro, U1 LT1762-3.3, U2 FT2232H, U3 93LC56-SO8, U4 CA25C1204GLT

Commit message: Schematic, PCB and BOM done.
Parts:
- removed D1: SMBJ6.0CA, ICE40PROG:DO_214AA, symbol Device:D_TVS
- J1: footprint Connector_PinSocket_2.54mm:PinSocket_2x05_P2.54mm_Horizontal -> Connector_PinSocket_2.54mm:PinSocket_2x05_P2.54mm_Vertical
- R7: renamed from R1; value 220 -> 270
- renumbered U4 to Q1, R2 to R1, R3 to R2, R4 to R3, R5 to R4, R6 to R5, R7 to R6
Other:
- moved on the sheet: C13, C14, C15, C16, C3, C4, C5, C6, C7, D2, FB1, J1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
